File: cosmic_watch_remix_V1/_autosave-cosmic_watch_remix_V1.kicad_sch (KiCad schematic)
At the start: 26 parts, among them IC1 MICROFJ-60035-TSV-TR1, IC2 LT3461AES6#TRMPBF, J1 Conn_01x05_Female, U1 ADS1115IDGS, U2 LM358

Commit message: V1.0
Finished Layout, Ready to Review!
Parts:
- added unit 1 of U2
- IC2: footprint Package_SO:SOIC-8-1EP_3.9x4.9mm_P1.27mm_EP2.29x3mm -> Package_TO_SOT_SMD:TSOT-23-6
- U2: footprint Package_SO:SOIC-8_7.5x5.85mm_P1.27mm -> Package_SO:SOIC-8-1EP_3.9x4.9mm_P1.27mm_EP2.29x3mm
Connections:
- net at D1.1 (A), R9.1: now also U2.3 (+)
- net at D1.2 (K), D2.1 (A): now also U2.1
- net at R8.2: now also U2.2 (-)
Changed lines of the file:
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@@
       (effects (font (size 1.27 1.27)) (justify left))
     )
-    (property "Footprint" "Package_SO:SOIC-8_7.5x5.85mm_P1.27mm" (id 2) (at 116.205 78.105 0)
+    (property "Footprint" "Package_SO:SOIC-8-1EP_3.9x4.9mm_P1.27mm_EP2.29x3mm" (id 2) (at 116.205 78.105 0)
       (effects (font (size 1.27 1.27)) hide)
     )
@@
     (pin "2")
   )
+  (symbol (lib_id "Amplifier_Operational:LM358") (at 133.35 90.805 0) (unit 1)
+    (in_bom yes) (on_board yes) (fields_autoplaced)
+    (property "Reference" "U2" (id 0) (at 133.35 82.0252 0))
+    (property "Value" "LM358" (id 1) (at 133.35 84.5621 0))
+    (property "Footprint" "Package_SO:SOIC-8-1EP_3.9x4.9mm_P1.27mm_EP2.29x3mm" (id 2) (at 133.35 90.805 0)
+      (effects (font (size 1.27 1.27)) hide)
+    )
+    (property "Datasheet" "http://www.ti.com/lit/ds/symlink/lm2904-n.pdf" (id 3) (at 133.35 90.805 0)
+      (effects (font (size 1.27 1.27)) hide)
+    )
+    (pin "1")
+    (pin "2")
+    (pin "3")
+  )
   (symbol (lib_id "power:GND") (at 182.88 104.14 0) (unit 1)
     (in_bom yes) (on_board yes) (fields_autoplaced)
@@
     (property "Reference" "IC2" (id 0) (at 47.625 33.181 0))
     (property "Value" "LT3461AES6#TRMPBF" (id 1) (at 47.625 35.7179 0))
-    (property "Footprint" "Package_SO:SOIC-8-1EP_3.9x4.9mm_P1.27mm_EP2.29x3mm" (id 2) (at 57.785 36.83 0)
+    (property "Footprint" "Package_TO_SOT_SMD:TSOT-23-6" (id 2) (at 57.785 36.83 0)
       (effects (font (size 1.27 1.27)) (justify left) hide)
     )
@@
     (property "Reference" "U2" (id 0) (at 164.465 79.4852 0))
     (property "Value" "LM358" (id 1) (at 164.465 82.0221 0))
-    (property "Footprint" "Package_SO:SOIC-8_7.5x5.85mm_P1.27mm" (id 2) (at 164.465 88.265 0)
+    (property "Footprint" "Package_SO:SOIC-8-1EP_3.9x4.9mm_P1.27mm_EP2.29x3mm" (id 2) (at 164.465 88.265 0)
       (effects (font (size 1.27 1.27)) hide)
     )
@@
     )
     (path "/4b58244c-d701-49ba-a686-6f48defc97f6"
-      (reference "IC2") (unit 1) (value "LT3461AES6#TRMPBF") (footprint "Package_SO:SOIC-8-1EP_3.9x4.9mm_P1.27mm_EP2.29x3mm")
+      (reference "IC2") (unit 1) (value "LT3461AES6#TRMPBF") (footprint "Package_TO_SOT_SMD:TSOT-23-6")
     )
     (path "/0a932650-28f5-47c0-b276-6314fc41caa3"
@@
       (reference "U1") (unit 1) (value "ADS1115IDGS") (footprint "Package_SO:TSSOP-10_3x3mm_P0.5mm")
     )
+    (path "/3d87b7d0-0327-4a61-b85c-7794ea82c7dd"
+      (reference "U2") (unit 1) (value "LM358") (footprint "Package_SO:SOIC-8-1EP_3.9x4.9mm_P1.27mm_EP2.29x3mm")
+    )
     (path "/a35a6c98-a3e9-4551-b1d6-01002dfe893f"
-      (reference "U2") (unit 2) (value "LM358") (footprint "Package_SO:SOIC-8_7.5x5.85mm_P1.27mm")
+      (reference "U2") (unit 2) (value "LM358") (footprint "Package_SO:SOIC-8-1EP_3.9x4.9mm_P1.27mm_EP2.29x3mm")
     )
     (path "/10a8a9c1-f318-4428-938d-d0192fe0148d"
-      (reference "U2") (unit 3) (value "LM358") (footprint "Package_SO:SOIC-8_7.5x5.85mm_P1.27mm")
-    )
-  )
+      (reference "U2") (unit 3) (value "LM358") (footprint "Package_SO:SOIC-8-1EP_3.9x4.9mm_P1.27mm_EP2.29x3mm")
+    )
+  )

Commit message: Completed Component Selection
Note change to 28V output
Parts:
- removed unit 1 of U2
- added U?: LM358, symbol Amplifier_Operational:LM358
- C9: value ? -> 22nF
- IC2: footprint Package_TO_SOT_SMD:TSOT-23-6 -> Package_SO:SOIC-8-1EP_3.9x4.9mm_P1.27mm_EP2.29x3mm
- R10: value ? -> 100k
- R6: value 280K -> 220K
- U2: footprint Package_SO:SOIC-8-1EP_3.9x4.9mm_P1.27mm_EP2.29x3mm -> Package_SO:SOIC-8_7.5x5.85mm_P1.27mm
Changed lines of the file:
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@@
   (junction (at 39.37 128.27) (diameter 0) (color 0 0 0 0)
   )
+  (junction (at 140.97 90.678) (diameter 0) (color 0 0 0 0)
+  )
   (junction (at 99.06 105.41) (diameter 0) (color 0 0 0 0)
   )
@@
   (junction (at 26.035 41.91) (diameter 0) (color 0 0 0 0)
   )
+  (junction (at 125.73 93.218) (diameter 0) (color 0 0 0 0)
+  )
   (junction (at 99.06 135.89) (diameter 0) (color 0 0 0 0)
   )
@@
   )
   (junction (at 33.655 26.67) (diameter 0) (color 0 0 0 0)
+  )
+  (junction (at 125.73 88.138) (diameter 0) (color 0 0 0 0)
   )
   (no_connect (at 192.405 90.805))
@@
       (effects (font (size 1.27 1.27)) (justify left))
     )
-    (property "Footprint" "Package_SO:SOIC-8-1EP_3.9x4.9mm_P1.27mm_EP2.29x3mm" (id 2) (at 116.205 78.105 0)
+    (property "Footprint" "Package_SO:SOIC-8_7.5x5.85mm_P1.27mm" (id 2) (at 116.205 78.105 0)
       (effects (font (size 1.27 1.27)) hide)
     )
@@
     (pin "2")
   )
-  (symbol (lib_id "Amplifier_Operational:LM358") (at 133.35 90.805 0) (unit 1)
-    (in_bom yes) (on_board yes) (fields_autoplaced)
-    (property "Reference" "U2" (id 0) (at 133.35 82.0252 0))
-    (property "Value" "LM358" (id 1) (at 133.35 84.5621 0))
-    (property "Footprint" "Package_SO:SOIC-8-1EP_3.9x4.9mm_P1.27mm_EP2.29x3mm" (id 2) (at 133.35 90.805 0)
-      (effects (font (size 1.27 1.27)) hide)
-    )
-    (property "Datasheet" "http://www.ti.com/lit/ds/symlink/lm2904-n.pdf" (id 3) (at 133.35 90.805 0)
+  (symbol (lib_id "Amplifier_Operational:LM358") (at 133.35 90.678 0) (unit 1)
+    (in_bom yes) (on_board yes) (fields_autoplaced)
+    (property "Reference" "U?" (id 0) (at 133.35 81.8982 0))
+    (property "Value" "LM358" (id 1) (at 133.35 84.4351 0))
+    (property "Footprint" "" (id 2) (at 133.35 90.678 0)
+      (effects (font (size 1.27 1.27)) hide)
+    )
+    (property "Datasheet" "http://www.ti.com/lit/ds/symlink/lm2904-n.pdf" (id 3) (at 133.35 90.678 0)
       (effects (font (size 1.27 1.27)) hide)
     )
@@
     (property "Reference" "IC2" (id 0) (at 47.625 33.181 0))
     (property "Value" "LT3461AES6#TRMPBF" (id 1) (at 47.625 35.7179 0))
-    (property "Footprint" "Package_TO_SOT_SMD:TSOT-23-6" (id 2) (at 57.785 36.83 0)
+    (property "Footprint" "Package_SO:SOIC-8-1EP_3.9x4.9mm_P1.27mm_EP2.29x3mm" (id 2) (at 57.785 36.83 0)
       (effects (font (size 1.27 1.27)) (justify left) hide)
     )
@@
     (in_bom yes) (on_board yes) (fields_autoplaced)
     (property "Reference" "R6" (id 0) (at 47.625 48.6242 90))
-    (property "Value" "280K" (id 1) (at 47.625 51.1611 90))
+    (property "Value" "220K" (id 1) (at 47.625 51.1611 90))
     (property "Footprint" "Resistor_SMD:R_0603_1608Metric" (id 2) (at 47.625 51.562 90)
       (effects (font (size 1.27 1.27)) hide)
@@
       (effects (font (size 1.27 1.27)) (justify left))
     )
-    (property "Value" "?" (id 1) (at 155.956 98.2222 0)
+    (property "Value" "22nF" (id 1) (at 155.956 98.2222 0)
       (effects (font (size 1.27 1.27)) (justify left))
     )
@@
     (property "Reference" "U2" (id 0) (at 164.465 79.4852 0))
     (property "Value" "LM358" (id 1) (at 164.465 82.0221 0))
-    (property "Footprint" "Package_SO:SOIC-8-1EP_3.9x4.9mm_P1.27mm_EP2.29x3mm" (id 2) (at 164.465 88.265 0)
+    (property "Footprint" "Package_SO:SOIC-8_7.5x5.85mm_P1.27mm" (id 2) (at 164.465 88.265 0)
       (effects (font (size 1.27 1.27)) hide)
     )
@@
   (symbol (lib_id "Device:R") (at 182.88 95.885 0) (mirror x) (unit 1)
     (in_bom yes) (on_board yes) (fields_autoplaced)
-    (property "Reference" "R10" (id 0) (at 181.102 95.0503 0)
+    (property "Reference" "R10" (id 0) (at 181.1021 95.0503 0)
       (effects (font (size 1.27 1.27)) (justify right))
     )
-    (property "Value" "?" (id 1) (at 181.102 97.5872 0)
+    (property "Value" "100k" (id 1) (at 181.1021 97.5872 0)
       (effects (font (size 1.27 1.27)) (justify right))
     )
@@
     )
     (path "/8d129ac0-21e8-4168-b5e8-555f7b81464d"
-      (reference "C9") (unit 1) (value "?") (footprint "Capacitor_SMD:C_0603_1608Metric")
+      (reference "C9") (unit 1) (value "22nF") (footprint "Capacitor_SMD:C_0603_1608Metric")
     )
     (path "/10789bbb-c1d1-4df2-bd22-ae0dfea0e3cd"
@@
     )
     (path "/4b58244c-d701-49ba-a686-6f48defc97f6"
-      (reference "IC2") (unit 1) (value "LT3461AES6#TRMPBF") (footprint "Package_TO_SOT_SMD:TSOT-23-6")
+      (reference "IC2") (unit 1) (value "LT3461AES6#TRMPBF") (footprint "Package_SO:SOIC-8-1EP_3.9x4.9mm_P1.27mm_EP2.29x3mm")
     )
     (path "/0a932650-28f5-47c0-b276-6314fc41caa3"
@@
     )
     (path "/8c8f7f6f-f151-43d0-b7c2-857bd66addff"
-      (reference "R6") (unit 1) (value "280K") (footprint "Resistor_SMD:R_0603_1608Metric")
+      (reference "R6") (unit 1) (value "220K") (footprint "Resistor_SMD:R_0603_1608Metric")
     )
     (path "/b047d4a8-77a5-43d5-bbbe-e454ef0e254d"
@@
     )
     (path "/a57db792-acd1-4a7c-9f3f-af8789d22ea8"
-      (reference "R10") (unit 1) (value "?") (footprint "Resistor_SMD:R_0603_1608Metric")
+      (reference "R10") (unit 1) (value "100k") (footprint "Resistor_SMD:R_0603_1608Metric")
     )
     (path "/d4e5a639-c802-4fd5-bd43-bd9483f1fee3"
       (reference "U1") (unit 1) (value "ADS1115IDGS") (footprint "Package_SO:TSSOP-10_3x3mm_P0.5mm")
     )
-    (path "/3d87b7d0-0327-4a61-b85c-7794ea82c7dd"
-      (reference "U2") (unit 1) (value "LM358") (footprint "Package_SO:SOIC-8-1EP_3.9x4.9mm_P1.27mm_EP2.29x3mm")
-    )
     (path "/a35a6c98-a3e9-4551-b1d6-01002dfe893f"
-      (reference "U2") (unit 2) (value "LM358") (footprint "Package_SO:SOIC-8-1EP_3.9x4.9mm_P1.27mm_EP2.29x3mm")
+      (reference "U2") (unit 2) (value "LM358") (footprint "Package_SO:SOIC-8_7.5x5.85mm_P1.27mm")
     )
     (path "/10a8a9c1-f318-4428-938d-d0192fe0148d"
-      (reference "U2") (unit 3) (value "LM358") (footprint "Package_SO:SOIC-8-1EP_3.9x4.9mm_P1.27mm_EP2.29x3mm")
-    )
-  )
+      (reference "U2") (unit 3) (value "LM358") (footprint "Package_SO:SOIC-8_7.5x5.85mm_P1.27mm")
+    )
+    (path "/2e435b0f-671e-4da0-9b1a-48c487e95e18"
+      (reference "U?") (unit 1) (value "LM358") (footprint "")
+    )
+  )
